File: charger.kicad_sch (KiCad schematic)
At the start: 3 parts

Commit message: buckboost: draft LM5176 4-switch power stage
Placed and wired the LM5176 (U1, HTSSOP-28-EP, LCSC C442493 per
TOPOLOGY.md) plus its support network:

Power stage: Q1..Q4 (30V/20A N-FET placeholder -- v1's FDS9926A is
undersized for v2's 5A/6.5A-peak spec, so this is marked TBD for a
proper JLCPCB Basic pick), L1 6.8uH, R8 5m current sense, boot caps
C5/C6 100nF, output caps C10/C11 22uF each.

Chip support: VIN caps C1/C2 22uF, VCC decoupling C3 2.2uF, BIAS C4
1uF, feedback R1/R2 (110k/10k -> 12.0V from LM5176's 1.0V Vref),
COMP R3 20k + C8 4.7nF, SS C7 10nF, RT R4 40.2k (~500kHz), EN
pull-up R6 100k to BAT+. MODE and DITH tied to GND.

Named nets wired: BAT+, GND, VOUT_12V, SW1, SW2, HDRV1/2, LDRV1/2,
BOOT1/2, FB, LM5176_VCC, LM5176_BIAS, SS, COMP, COMP_MID, RT, EN.
No hierarchical sheet pins -- power rails cross sheets via global
labels per the root-sheet plan.

TBD annotation on-sheet lists what needs a review pass: FET MPN,
CS/CSG hookup (currently unconnected -- either wire R8 across L1 as
high-side inductor sense OR switch to Rds(on) sensing on Q2/Q3),
SLOPE resistor R5 sizing, and optional PGOOD LED.

Also cleaned the three TEMPLATE_R/C/D placeholder symbols that
create_schematic left in all four sub-sheets.

Co-Authored-By: Claude Opus 4.7 <noreply@anthropic.com>
Parts:
- removed _TEMPLATE_C: C_TEMPLATE, symbol Device:C
- removed _TEMPLATE_D: LED_TEMPLATE, symbol Device:LED
- removed _TEMPLATE_R: R_TEMPLATE, symbol Device:R

Commit message: charger: draft IP2326 + support network sheet
19 components: IP2326 (VQFN-24, LCSC C2832094), 2.2 µH boost inductor,
Cin/Csys/Cout ceramics, bootstrap cap, CON_SEL pull-down (1 kΩ → 3S mode),
NTC divider, charge LED + series R, VSET/UVSET/OVSET/TIME_SET/ISET/EN
config resistors. Pins 1/2 (D+/D-) and 23/24 (VBATM/VBAT_GND) marked NC
so PD negotiation goes through CH224K on the input sheet and BQ76920
handles all cell balancing.

Cross-sheet nets exported as globals: VBUS_9V (from input), BAT+ (to bms
and buckboost), GND. ERC clean apart from cosmetic Unspecified/Passive
pin-type warnings from the IP2326 library symbol.

Co-Authored-By: Claude Opus 4.7 <noreply@anthropic.com>
Parts:
- added C1, C4: 10uF, symbol Device:C
- added C2, C3: 22uF, symbol Device:C
- added C5: 100nF, symbol Device:C
- added D1: LED_CHG, symbol Device:LED
- added L1: 2.2uH, symbol Device:L
- added R1, R2, R3, R8: 10k, symbol Device:R
- added R10: 4.7k, symbol Device:R
- added R4, R5, R6, R9: 100k, symbol Device:R
- added R7: 1k, symbol Device:R
- added TH1: 10k NTC, symbol Device:Thermistor_NTC
- added U1: IP2326, symbol power_module_lib:IP2326
Connections:
- new net BAT+: C4.1, U1.21 (VOUT), U1.22 (VOUT)
- new net BAT_STAT: R3.2, U1.5 (BAT_STAT)
- new net BST_CAP: C5.1, U1.14 (BST)
- new net CON_SEL: R7.1, U1.10 (CON_SEL)
- new net EN: R9.2, U1.12 (EN)
- new net GND: C1.2, C2.2, C3.2, C4.2, R1.2, R4.2, R5.2, R6.2, R7.2, R8.2, TH1.2, U1.18 (PGND), U1.25 (EP)
- new net ISET: R8.1, U1.11 (ISET)
- new net LED_K: R10.2, U1.6 (LED)
- new net LED_MID: D1.1 (K), R10.1
- new net LX_SW: C5.2, L1.2, U1.15 (LX), U1.16 (LX), U1.17 (LX)
- new net NTC_MID: R2.2, TH1.1, U1.4 (NTC)
- new net TIME_SET: R4.1, U1.7 (TIME_SET)
- new net VBUS_9V: C1.1, L1.1, R9.1, U1.13 (VIN)
- new net VIN_OVSET: R6.1, U1.9 (VIN_OVSET)
- new net VIN_UVSET: R5.1, U1.8 (VIN_UVSET)
- new net VSET: R1.1, U1.3 (VSET)
- new net VSYS: C2.1, C3.1, D1.2 (A), R2.1, R3.1, U1.19 (VSYS), U1.20 (VSYS)
- no-connect marks 0 -> 4
