File: input.kicad_sch (KiCad schematic)
At the start: 3 parts

Commit message: buckboost: draft LM5176 4-switch power stage
Placed and wired the LM5176 (U1, HTSSOP-28-EP, LCSC C442493 per
TOPOLOGY.md) plus its support network:

Power stage: Q1..Q4 (30V/20A N-FET placeholder -- v1's FDS9926A is
undersized for v2's 5A/6.5A-peak spec, so this is marked TBD for a
proper JLCPCB Basic pick), L1 6.8uH, R8 5m current sense, boot caps
C5/C6 100nF, output caps C10/C11 22uF each.

Chip support: VIN caps C1/C2 22uF, VCC decoupling C3 2.2uF, BIAS C4
1uF, feedback R1/R2 (110k/10k -> 12.0V from LM5176's 1.0V Vref),
COMP R3 20k + C8 4.7nF, SS C7 10nF, RT R4 40.2k (~500kHz), EN
pull-up R6 100k to BAT+. MODE and DITH tied to GND.

Named nets wired: BAT+, GND, VOUT_12V, SW1, SW2, HDRV1/2, LDRV1/2,
BOOT1/2, FB, LM5176_VCC, LM5176_BIAS, SS, COMP, COMP_MID, RT, EN.
No hierarchical sheet pins -- power rails cross sheets via global
labels per the root-sheet plan.

TBD annotation on-sheet lists what needs a review pass: FET MPN,
CS/CSG hookup (currently unconnected -- either wire R8 across L1 as
high-side inductor sense OR switch to Rds(on) sensing on Q2/Q3),
SLOPE resistor R5 sizing, and optional PGOOD LED.

Also cleaned the three TEMPLATE_R/C/D placeholder symbols that
create_schematic left in all four sub-sheets.

Co-Authored-By: Claude Opus 4.7 <noreply@anthropic.com>
Parts:
- removed _TEMPLATE_C: C_TEMPLATE, symbol Device:C
- removed _TEMPLATE_D: LED_TEMPLATE, symbol Device:LED
- removed _TEMPLATE_R: R_TEMPLATE, symbol Device:R

Commit message: input: draft USB-C + CH224K + input protection sheet; add BAT+/VBUS_9V PWR_FLAGs
input.kicad_sch (8 functional + 2 PWR_FLAG for ERC): 16-pin USB-C
receptacle (charge-only — D+/D-, SBU1/2 all NC), CH224K PD sink
controller strapped for 9V PDO via 24k CFG1→GND, SRV05-4 ESD array on
CC1/CC2, SMAJ12A TVS on VBUS_RAW, 600Ω@100MHz ferrite between VBUS_RAW
and VBUS_9V, plus 10 µF caps on both sides.

Sheet ERC clean (0 err / 2 warn, both local↔global label pairs, which
are the intentional cross-sheet plumbing).

Also added PWR_FLAG on bms.BAT+ so the cross-sheet ERC recognises the
pack rail as a driven power source.

Co-Authored-By: Claude Opus 4.7 <noreply@anthropic.com>
Parts:
- added C1, C2: 10uF, symbol Device:C
- added D1: SRV05-4, symbol Power_Protection:SRV05-4
- added D2: SMAJ12A, symbol Device:D_TVS
- added FB1: 600R@100MHz, symbol Device:FerriteBead
- added J1: USB_C_16P, symbol Connector:USB_C_Receptacle_USB2.0_16P
- added R1: 24k, symbol Device:R
- added U1: CH224K, symbol Interface_USB:CH224K
Connections:
- new net CC1: D1.1 (IO1), J1.A5 (CC1), U1.7 (CC1)
- new net CC2: D1.3 (IO2), J1.B5 (CC2), U1.6 (CC2)
- new net CFG1_SEL: R1.1, U1.9 (CFG1)
- new net GND: C1.2, C2.2, D1.2 (VN), D2.2 (A2), J1.A1 (GND), J1.A12 (GND), J1.B1 (GND), J1.B12 (GND), J1.S1 (SHIELD), R1.2, U1.11 (GND)
- new net VBUS_9V: C2.1, FB1.2
- new net VBUS_RAW: C1.1, D1.5 (VP), D2.1 (A1), FB1.1, J1.A4 (VBUS), J1.A9 (VBUS), J1.B4 (VBUS), J1.B9 (VBUS), U1.1 (VDD), U1.8 (VBUS)
- no-connect marks 0 -> 13
