File: power_module_v2alt.kicad_pcb (KiCad board)
At the start: 2 copper layers, 0 parts

Commit message: Step 2: complete Footprint set + sync 76 footprints to .kicad_pcb
Fill in the Footprint properties that were missing from the prior
sourcing pass, and sync everything to the PCB.

Footprint updates on the schematic:
- 35 passives got their Footprint assigned by value (0603 for R/C ≤1uF,
  0805 for 10uF/22uF caps).
- BAT1_BMS1 → power_module_lib:BAT-SMD_BH-18650-B5BA016 (was truncated).
- L1_BUCKBOOST1 → Inductor_SMD:L_Sumida_CDMC6D28_7.25x6.5mm (needed the
  size suffix so KiCad can resolve the .kicad_mod file).

Sync result: 76/76 footprints imported, 60 nets added, 245 pads assigned,
0 import errors.  Unmatched pads reported are all intentional NCs per
REQUIREMENTS.md (USB-C D+/D-, CH224K SBU/CFG, SRV05-4 unused ESD channels).

The footprints are at the default y=-140..-20 auto-import grid; no
placement work yet.  Next step is add_board_outline + set_design_rules.

For discoverability going forward, the pre-sync gap gets caught by
check_sourcing_readiness (KiCAD-MCP-Server fa93ba9 on develop) rather
than having to reset the .kicad_pcb after every retro-fill of an empty
Footprint property.

Co-Authored-By: Claude Opus 4.7 <noreply@anthropic.com>
Parts:
- added BAT1_BMS1: BH-18650-B5BA016, power_module_lib:BAT-SMD_BH-18650-B5BA016, F.Cu at (20.0, -20.0)
- added C10_BUCKBOOST1: 22uF, Capacitor_SMD:C_0805_2012Metric, F.Cu at (5.00, -155.0)
- added C11_BUCKBOOST1: 22uF, Capacitor_SMD:C_0805_2012Metric, F.Cu at (20.0, -155.0)
- added C1_BMS1: 100nF, Capacitor_SMD:C_0603_1608Metric, F.Cu at (20.0, -35.0)
- added C1_BUCKBOOST1: 22uF, Capacitor_SMD:C_0805_2012Metric, F.Cu at (65.0, -110.0)
- added C1_CHARGER1: 10uF, Capacitor_SMD:C_0805_2012Metric, F.Cu at (20.0, -170.0)
- added C1_INPUT1: 10uF, Capacitor_SMD:C_0805_2012Metric, F.Cu at (50.0, -230.0)
- added C2_BMS1: 100nF, Capacitor_SMD:C_0603_1608Metric, F.Cu at (35.0, -35.0)
- added C2_BUCKBOOST1: 22uF, Capacitor_SMD:C_0805_2012Metric, F.Cu at (5.00, -125.0)
- added C2_CHARGER1: 22uF, Capacitor_SMD:C_0805_2012Metric, F.Cu at (35.0, -170.0)
- added C2_INPUT1: 10uF, Capacitor_SMD:C_0805_2012Metric, F.Cu at (65.0, -230.0)
- added C3_BMS1: 100nF, Capacitor_SMD:C_0603_1608Metric, F.Cu at (50.0, -35.0)
- added C3_BUCKBOOST1: 2.2uF, Capacitor_SMD:C_0603_1608Metric, F.Cu at (20.0, -125.0)
- added C3_CHARGER1: 22uF, Capacitor_SMD:C_0805_2012Metric, F.Cu at (50.0, -170.0)
- added C4_BMS1: 100nF, Capacitor_SMD:C_0603_1608Metric, F.Cu at (65.0, -35.0)
- added C4_BUCKBOOST1: 1uF, Capacitor_SMD:C_0603_1608Metric, F.Cu at (35.0, -125.0)
- added C4_CHARGER1: 10uF, Capacitor_SMD:C_0805_2012Metric, F.Cu at (65.0, -170.0)
- added C5_BMS1: 1uF, Capacitor_SMD:C_0603_1608Metric, F.Cu at (50.0, -50.0)
- added C5_BUCKBOOST1: 100nF, Capacitor_SMD:C_0603_1608Metric, F.Cu at (50.0, -125.0)
- added C5_CHARGER1: 100nF, Capacitor_SMD:C_0603_1608Metric, F.Cu at (5.00, -185.0)
- added C6_BMS1: 100nF, Capacitor_SMD:C_0603_1608Metric, F.Cu at (65.0, -50.0)
- added C6_BUCKBOOST1: 100nF, Capacitor_SMD:C_0603_1608Metric, F.Cu at (65.0, -125.0)
- added C7_BMS1: 1uF, Capacitor_SMD:C_0603_1608Metric, F.Cu at (5.00, -65.0)
- added C7_BUCKBOOST1: 10nF, Capacitor_SMD:C_0603_1608Metric, F.Cu at (65.0, -95.0)
- added C8_BUCKBOOST1: 4.7nF, Capacitor_SMD:C_0603_1608Metric, F.Cu at (50.0, -110.0)
- added D1_BMS1: SMAJ15A, Diode_SMD:D_SMA, F.Cu at (5.00, -50.0)
- added D1_CHARGER1: LED_CHG (Red), LED_SMD:LED_0603_1608Metric, F.Cu at (5.00, -200.0)
- added D1_INPUT1: SRV05-4, Package_TO_SOT_SMD:SOT-23-6, F.Cu at (5.00, -230.0)
- added D2_BMS1: SMAJ15A, Diode_SMD:D_SMA, F.Cu at (20.0, -50.0)
- added D2_INPUT1: SMAJ12A, Diode_SMD:D_SMA, F.Cu at (20.0, -230.0)
- added D3_BMS1: SMAJ15A, Diode_SMD:D_SMA, F.Cu at (35.0, -50.0)
- added FB1_INPUT1: 600R@100MHz, Inductor_SMD:L_0603_1608Metric, F.Cu at (35.0, -230.0)
- added J1_BMS1: I2C+ALERT, Connector_PinHeader_2.54mm:PinHeader_1x05_P2.54mm_Vertical, F.Cu at (20.0, -80.0)
- added J1_INPUT1: USB_C_16P, Connector_USB:USB_C_Receptacle_HRO_TYPE-C-31-M-12, F.Cu at (50.0, -215.0)
- added L1_BUCKBOOST1: 6.8uH, Inductor_SMD:L_Sumida_CDMC6D28_7.25x6.5mm, F.Cu at (65.0, -140.0)
- added L1_CHARGER1: 2.2uH, Inductor_SMD:L_Sunlord_MWSA0402S, F.Cu at (5.00, -170.0)
- added Q1_BMS1: AON7544, power_module_lib:DFN-8_L3.3-W3.3-P0.65-BL-2, F.Cu at (50.0, -80.0)
- added Q1_BUCKBOOST1: AON7544, power_module_lib:DFN-8_L3.3-W3.3-P0.65-BL-2, F.Cu at (5.00, -140.0)
- added Q2_BMS1: AON7544, power_module_lib:DFN-8_L3.3-W3.3-P0.65-BL-2, F.Cu at (65.0, -80.0)
- added Q2_BUCKBOOST1: AON7544, power_module_lib:DFN-8_L3.3-W3.3-P0.65-BL-2, F.Cu at (20.0, -140.0)
- added Q3_BUCKBOOST1: AON7544, power_module_lib:DFN-8_L3.3-W3.3-P0.65-BL-2, F.Cu at (35.0, -140.0)
- added Q4_BUCKBOOST1: AON7544, power_module_lib:DFN-8_L3.3-W3.3-P0.65-BL-2, F.Cu at (50.0, -140.0)
- added R10_BMS1: 100, Resistor_SMD:R_0603_1608Metric, F.Cu at (5.00, -95.0)
- added R10_CHARGER1: 4.7k, Resistor_SMD:R_0603_1608Metric, F.Cu at (20.0, -200.0)
- added R11_BMS1: 100, Resistor_SMD:R_0603_1608Metric, F.Cu at (20.0, -95.0)
- added R1_BMS1: 100, Resistor_SMD:R_0603_1608Metric, F.Cu at (35.0, -20.0)
- added R1_BUCKBOOST1: 110k, Resistor_SMD:R_0603_1608Metric, F.Cu at (35.0, -155.0)
- added R1_CHARGER1: 100k, Resistor_SMD:R_0603_1608Metric, F.Cu at (20.0, -185.0)
- added R1_INPUT1: 24k, Resistor_SMD:R_0603_1608Metric, F.Cu at (5.00, -245.0)
- added R2_BMS1: 100, Resistor_SMD:R_0603_1608Metric, F.Cu at (50.0, -20.0)
- added R2_BUCKBOOST1: 10k, Resistor_SMD:R_0603_1608Metric, F.Cu at (50.0, -155.0)
- added R2_CHARGER1: 10k, Resistor_SMD:R_0603_1608Metric, F.Cu at (35.0, -185.0)
- added R3_BMS1: 100, Resistor_SMD:R_0603_1608Metric, F.Cu at (65.0, -20.0)
- added R3_BUCKBOOST1: 20k, Resistor_SMD:R_0603_1608Metric, F.Cu at (35.0, -110.0)
- added R3_CHARGER1: 10k, Resistor_SMD:R_0603_1608Metric, F.Cu at (65.0, -185.0)
- added R4_BMS1: 100, Resistor_SMD:R_0603_1608Metric, F.Cu at (5.00, -35.0)
- added R4_BUCKBOOST1: 40.2k, Resistor_SMD:R_0603_1608Metric, F.Cu at (5.00, -110.0)
- added R4_CHARGER1: 100k, Resistor_SMD:R_0603_1608Metric, F.Cu at (35.0, -200.0)
- added R5_BMS1: 10k, Resistor_SMD:R_0603_1608Metric, F.Cu at (20.0, -65.0)
- added R5_BUCKBOOST1: 20k, Resistor_SMD:R_0603_1608Metric, F.Cu at (20.0, -110.0)
- added R5_CHARGER1: 100k, Resistor_SMD:R_0603_1608Metric, F.Cu at (50.0, -200.0)
- added R6_BMS1: 10k, Resistor_SMD:R_0603_1608Metric, F.Cu at (35.0, -65.0)
- added R6_BUCKBOOST1: 100k, Resistor_SMD:R_0603_1608Metric, F.Cu at (50.0, -95.0)
- added R6_CHARGER1: 100k, Resistor_SMD:R_0603_1608Metric, F.Cu at (65.0, -200.0)
- added R7_BMS1: 10k, Resistor_SMD:R_0603_1608Metric, F.Cu at (50.0, -65.0)
- added R7_CHARGER1: 1k, Resistor_SMD:R_0603_1608Metric, F.Cu at (5.00, -215.0)
- added R8_BMS1: 10k, Resistor_SMD:R_0603_1608Metric, F.Cu at (65.0, -65.0)
- added R8_CHARGER1: 33k, Resistor_SMD:R_0603_1608Metric, F.Cu at (20.0, -215.0)
- added R9_BMS1: 5m, Resistor_SMD:R_2512_6332Metric, F.Cu at (35.0, -80.0)
- added R9_CHARGER1: 100k, Resistor_SMD:R_0603_1608Metric, F.Cu at (35.0, -215.0)
- added TH1_BMS1: 10k NTC (103AT), Resistor_SMD:R_0603_1608Metric, F.Cu at (5.00, -80.0)
- added TH1_CHARGER1: 10k NTC, Resistor_SMD:R_0603_1608Metric, F.Cu at (50.0, -185.0)
- added U1_BMS1: BQ7692003PWR, Package_SO:TSSOP-20_4.4x6.5mm_P0.65mm, F.Cu at (5.00, -20.0)
- added U1_BUCKBOOST1: LM5176PWP, Package_SO:HTSSOP-28-1EP_4.4x9.7mm_P0.65mm_EP3.4x9.5mm_ThermalVias, F.Cu at (35.0, -95.0)
- added U1_CHARGER1: IP2326, power_module_lib:VQFN-24_L4.0-W4.0-P0.50-BL-EP2.5, F.Cu at (65.0, -155.0)
- added U1_INPUT1: CH224K, Package_SO:SSOP-10-1EP_3.9x4.9mm_P1mm_EP2.1x3.3mm, F.Cu at (65.0, -215.0)

Commit message: Step 3+4 WIP: board outline, 4-layer stackup, decoupling spring classes, initial placement pass
Step 3 (board mechanics)
- Edge.Cuts rectangle 100x70 mm (BAT1 alone is 82.3x56.8 so 60x80 in
  the pre-session NOTES was too small)
- 4-layer stackup: added In1.Cu (GND plane) + In2.Cu (PWR plane)
- Design rules tightened: clearance 0.15, minTrackWidth 0.15,
  minViaDiameter 0.45, viaDrill 0.3

Step 4 (WIP — placement)
- 13 Pin_Spring_Class:{pad} = {"IC.pin": "DECOUPLING"} assignments on
  bypass caps across bms/charger/buckboost.  Every IC's power/reservoir/
  bootstrap cap now has an explicit DECOUPLING target so the auto-placer
  parks it right next to the IC pin instead of drifting off with the
  power-rail centroid:
    C7_BMS1        -> BQ76920 CAP1 (pin 7, charge pump reservoir)
    C5_BMS1        -> BQ76920 REGOUT bypass (pin 8)
    C6_BMS1        -> BQ76920 BAT+ sense
    C1..C4_BMS1    -> BQ76920 VCn sense RC filters
    C3_BUCKBOOST1  -> LM5176 BIAS bypass (pin 24, 2.2uF)
    C4_BUCKBOOST1  -> LM5176 VCC LDO bypass (pin 23, 1uF)
    C5_BUCKBOOST1  -> LM5176 BOOT1 bootstrap (pin 26)
    C6_BUCKBOOST1  -> LM5176 BOOT2 bootstrap (pin 20)
    C7_BUCKBOOST1  -> LM5176 SS (pin 8)
    C5_CHARGER1    -> IP2326 BST_CAP (pin 14)
- Initial relax_placement pass with 7 locked anchors (2 headers + BAT1 +
  4 ICs).  Not a shippable layout yet: USB-C is backwards, I2C header
  overlaps BAT1's B.Cu pad zone, Q1..Q4 + L1 (buck-boost power stage)
  scattered from LM5176.  Left as a starting point for hand-refinement.
- TH1_BMS1 (pack thermistor) flipped to B.Cu for proximity to the
  cells — final position to be set by hand.

Co-Authored-By: Claude Opus 4.7 <noreply@anthropic.com>
Parts:
- BAT1_BMS1, TH1_BMS1: moved to B.Cu
- moved R1_INPUT1 254.4 mm to (39.5, 7.04)
- moved C2_INPUT1 244.2 mm to (43.6, 13.2), turned to -90 degrees
- moved D1_INPUT1 235.6 mm to (26.5, 4.64), turned to 90 degrees
- moved C1_INPUT1 233.8 mm to (31.2, 3.05)
- moved R9_CHARGER1 233.5 mm to (46.6, 18.2), turned to -90 degrees
- moved FB1_INPUT1 233.2 mm to (36.9, 3.23)
- moved D2_INPUT1 232.9 mm to (28.6, 2.69), turned to 90 degrees
- moved R7_CHARGER1 231.4 mm to (59.8, 9.84)
- moved U1_INPUT1 225.3 mm to (33.0, 8.00)
- moved R8_CHARGER1 223.4 mm to (57.6, 5.21), turned to 90 degrees
- moved J1_INPUT1 222.0 mm to (20.0, 5.00)
- moved C10_BUCKBOOST1 221.3 mm to (42.0, 63.2), turned to -90 degrees
- moved C11_BUCKBOOST1 217.9 mm to (38.7, 62.1), turned to -90 degrees
- moved R10_CHARGER1 217.9 mm to (50.3, 15.7)
- moved D1_CHARGER1 217.5 mm to (46.7, 13.5), turned to 90 degrees
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Other:
- board outline added: 100 x 70 mm
- copper layers 2 -> 4
