File: power_module_v2alt.kicad_pcb (KiCad board)
At the start: 4 copper layers, 100 x 70 mm, 76 parts, among them J1_BMS1 I2C+ALERT, J1_INPUT1 USB_C_16P, Q1_BMS1 AON7544, Q1_BUCKBOOST1 AON7544, Q2_BMS1 AON7544, Q2_BUCKBOOST1 AON7544, Q3_BUCKBOOST1 AON7544, Q4_BUCKBOOST1 AON7544, U1_BMS1 BQ7692003PWR, U1_BUCKBOOST1 LM5176PWP, U1_CHARGER1 IP2326, U1_INPUT1 CH224K

Commit message: Adjusted locations of some components
Parts:
- moved J1_BMS1 41.4 mm to (75.9, 66.8), turned to 90 degrees
- moved J1_INPUT1 0.73 mm to (20.0, 4.27), turned to 180 degrees
