File: power_module_v2alt.kicad_pcb (KiCad board)
At the start: 4 copper layers, 100 x 70 mm, 77 parts, among them J1_BMS1 I2C+ALERT, J1_INPUT1 USB_C_16P, Q1_BMS1 AON7544, Q1_BUCKBOOST1 AON7544, Q2_BMS1 AON7544, Q2_BUCKBOOST1 AON7544, Q3_BUCKBOOST1 AON7544, Q4_BUCKBOOST1 AON7544, SW1_BMS1 Kill Switch, U1_BMS1 BQ7692003PWR, U1_BUCKBOOST1 LM5176PWP, U1_CHARGER1 IP2326, U1_INPUT1 CH224K

Commit message: Adjusted some positions
Parts:
- moved C1_BUCKBOOST1 40.8 mm to (49.5, 74.0), turned to 180 degrees
- moved C11_BUCKBOOST1 38.1 mm to (13.5, 74.0), turned to 180 degrees
- moved C2_BUCKBOOST1 37.6 mm to (49.5, 67.0), turned to 180 degrees
- moved C10_BUCKBOOST1 34.6 mm to (13.5, 67.0), turned to 180 degrees
- moved Q1_BUCKBOOST1 33.7 mm to (43.5, 77.0), turned to 180 degrees
- moved R4_BUCKBOOST1 32.4 mm to (34.5, 81.8), turned to -90 degrees
- moved Q4_BUCKBOOST1 31.5 mm to (19.5, 77.0), turned to 180 degrees
- moved C5_BUCKBOOST1 30.0 mm to (30.7, 81.0), turned to 0 degrees
- moved C8_BUCKBOOST1 27.8 mm to (39.7, 76.7), turned to -90 degrees
- moved Q2_BUCKBOOST1 27.4 mm to (43.5, 71.0), turned to 180 degrees
- moved R5_BUCKBOOST1 25.0 mm to (37.0, 76.8), turned to -90 degrees
- moved Q3_BUCKBOOST1 24.6 mm to (19.5, 71.0), turned to 180 degrees
- moved C3_BUCKBOOST1 24.4 mm to (25.4, 77.0), turned to 180 degrees
- moved C7_BUCKBOOST1 20.3 mm to (37.6, 73.5), turned to 0 degrees
- moved C4_BUCKBOOST1 19.9 mm to (25.4, 74.4), turned to 180 degrees
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Other:
- board size 100 x 70 mm -> 100 x 85 mm
