File: power_module_v2alt.kicad_pcb (KiCad board)
At the start: 4 copper layers, 100 x 85 mm, 77 parts, among them J1_BMS1 I2C+ALERT, J1_INPUT1 USB_C_16P, Q1_BMS1 AON7544, Q1_BUCKBOOST1 AON7544, Q2_BMS1 AON7544, Q2_BUCKBOOST1 AON7544, Q3_BUCKBOOST1 AON7544, Q4_BUCKBOOST1 AON7544, SW1_BMS1 Kill Switch, U1_BMS1 BQ7692003PWR, U1_BUCKBOOST1 LM5176PWP, U1_CHARGER1 IP2326, U1_INPUT1 CH224K

Commit message: Fix EN cross-sheet collision + tag charger VSYS/BAT decoupling caps
EN was accidentally shared across charger and buckboost

Both sheets carried a local label named "EN" — kicad-cli sch export
netlist correctly namespaces these as /charger/EN and /buckboost/EN, but
the .kicad_pcb had ONE net "EN" (net 42) with all four pads collapsed
into it: IP2326 pin 11 was electrically tied to LM5176 pin 1 through PCB
copper.  IP2326.EN is pulled up to VBUS_9V via R9_CHARGER1 (9V rail),
LM5176.EN is pulled up to BAT+ via R6_BUCKBOOST1 (12V rail); shorting
them would fight the pull-ups and give indeterminate enable behaviour.

Renamed the labels to make them unambiguously distinct:

  charger:   EN → CHG_EN
  buckboost: EN → BB_EN

Post-sync verification:
  EN     — 0 pads
  CHG_EN — R9_CHARGER1.2, U1_CHARGER1.11
  BB_EN  — R6_BUCKBOOST1.1, U1_BUCKBOOST1.1

Underlying sync_schematic_to_board bug (collapsing same-named local
labels across sheets when the kicad-cli netlist keeps them separate) is
filed for follow-up on the MCP-server side.  Sweep for other cross-sheet
collisions: only VBUS_9V (input↔charger, intentional) was found.

C2/C3/C4_CHARGER1 decoupling tags added

The earlier decoupling analyser only spotted caps whose non-power pad
lands on a *single* IC pin AND whose ground pad is literal "GND".  It
missed:

  C2_CHARGER1 (22uF) — VSYS bulk cap → tag DECOUPLING to U1_CHARGER1.19
  C3_CHARGER1 (22uF) — VSYS bulk cap → tag DECOUPLING to U1_CHARGER1.20
  C4_CHARGER1 (10uF) — BAT+ input cap → tag DECOUPLING to U1_CHARGER1.21

Distributes across VSYS pins 19+20 so the two 22uF caps don't fight for
the same target pin.  C4 was floating in the last relax pass because its
BAT+ pad was PLANE-classified (via META1 singleton) and GND is a
44-node auto-PLANE; explicit DECOUPLING gives it a target to anchor to.

Co-Authored-By: Claude Opus 4.7 <noreply@anthropic.com>
Connections:
- R6_BUCKBOOST1 pad 1: EN -> BB_EN
- R9_CHARGER1 pad 2: EN -> CHG_EN
- U1_BUCKBOOST1 pad 1: EN -> BB_EN
- U1_CHARGER1 pad 12: EN -> CHG_EN
