File: power_module_v2alt.kicad_pcb (KiCad board)
At the start: 4 copper layers, 100 x 85 mm, 77 parts, among them J1_BMS1 I2C+ALERT, J1_INPUT1 USB_C_16P, Q1_BMS1 AON7544, Q1_BUCKBOOST1 AON7544, Q2_BMS1 AON7544, Q2_BUCKBOOST1 AON7544, Q3_BUCKBOOST1 AON7544, Q4_BUCKBOOST1 AON7544, SW1_BMS1 Kill Switch, U1_BMS1 BQ7692003PWR, U1_BUCKBOOST1 LM5176PWP, U1_CHARGER1 IP2326, U1_INPUT1 CH224K

Commit message: A few position tweaks
Parts:
- moved C4_CHARGER1 46.2 mm to (50.0, 10.9), turned to 180 degrees
- moved R6_BUCKBOOST1 34.5 mm to (41.1, 67.8), turned to 90 degrees
- moved R9_CHARGER1 31.1 mm to (64.2, 7.37), turned to 180 degrees
- moved Q1_BMS1 3.50 mm to (84.1, 23.9)
- moved Q2_BMS1 3.50 mm to (84.0, 17.5)
- moved C2_CHARGER1 2.14 mm to (50.0, 8.19), turned to 180 degrees
- moved R6_CHARGER1 2.00 mm to (61.9, 9.14)
