File: power_module_v2alt.kicad_pcb (KiCad board)
At the start: 4 copper layers, 100 x 85 mm, 77 parts, among them J1_BMS1 I2C+ALERT, J1_INPUT1 USB_C_16P, Q1_BMS1 AON7544, Q1_BUCKBOOST1 AON7544, Q2_BMS1 AON7544, Q2_BUCKBOOST1 AON7544, Q3_BUCKBOOST1 AON7544, Q4_BUCKBOOST1 AON7544, SW1_BMS1 Kill Switch, U1_BMS1 BQ7692003PWR, U1_BUCKBOOST1 LM5176PWP, U1_CHARGER1 IP2326, U1_INPUT1 CH224K

Commit message: Step 5: pre-route audit + same-net zones + plane pours
Netclasses + patterns
- POWER_5A (1.65 mm track, 0.8/0.4 via) — BAT+, VOUT_12V
- POWER_2A (0.60 mm track, 0.6/0.3 via) — VBUS_RAW, VBUS_9V, VSYS
- mcp_expected_netclass_patterns authored on META1 singleton for
  drift protection.

Stale-net merges (sync_schematic_to_board leftovers)
- Net-(C6_BUCKBOOST1-Pad2) → SW2  (6 pads incl. Q4.S ×3, L1.pad2)
- Net-(U1_BMS1-Pad6)       → TS1  (BQ76920.6, R8.2, TH1.1)
These were both labelled correctly in the schematic; the PCB had
stale auto-names from an earlier state that later syncs never
migrated.  Same class of bug as the EN cross-sheet issue —
sync_schematic_to_board doesn't fully update net names once a net is
created.  Merged in .kicad_pcb via search-and-repoint script; net
numbering preserved so no downstream references break.

pin_zone_same_net (22 applied, 6 rejected)
- Q1..Q4 FET Source triplets (VSS / GND / SW1 / SW2)
- BQ76920 BAT+ pin pair (9+10)
- LM5176 EP thermal pad (pin 29) — 34.9 mm² GND cluster on B.Cu
- IP2326 VSYS pin pair (19+20) and BAT+ pin pair (21+22)
- USB-C shield pads (S1 pair)
- Rejections all valid (would overlap foreign pads on connectors
  and the LM5176 body).

Plane pours
- In1.Cu = GND across full board outline (0.5 mm inset)
- In2.Cu = BAT+ across full board outline
- VOUT_12V will route as short traces on F.Cu/B.Cu from LM5176's
  output pins to the C10/C11 output caps — the net is local and
  doesn't need its own plane.

pre_route_audit: 66 → 7 unreachable spokes after pours
- 5 LM5176 comp-loop signals (FB / RT / COMP / SLOPE / SS) that
  the audit can't route at netclass width because the LM5176 body
  blocks the direct F.Cu path; freerouting will handle with short
  hops.
- 2 BAT+ BAT1.1 → IP2326.21/22: spoke_no_anchor is a tool artifact
  for BAT1's large custom B.Cu pads (the audit can't find a
  representative anchor point on a 41×18 mm pad).  In practice the
  BAT+ plane on In2.Cu will thermal-connect BAT1 to the charger via
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
Connections:
- net Net-(U1_BMS1-Pad6) renamed TS1
- C6_BUCKBOOST1 pad 2: Net-(C6_BUCKBOOST1-Pad2) -> SW2
- L1_BUCKBOOST1 pad 2: Net-(C6_BUCKBOOST1-Pad2) -> SW2
- Q3_BUCKBOOST1 pad D: Net-(C6_BUCKBOOST1-Pad2) -> SW2
- Q4_BUCKBOOST1 pad S: Net-(C6_BUCKBOOST1-Pad2) -> SW2
Routing:
- added copper zone on F.Cu, net BAT+
- added copper zone on In2.Cu, net BAT+
- added copper zone on B.Cu, net GND
- added copper zone on F.Cu, net GND
- added copper zone on In1.Cu, net GND
- added copper zone on F.Cu, net LX_SW
- added copper zone on F.Cu, net SW1
- added copper zone on F.Cu, net SW2
- added copper zone on F.Cu, net VC3
- added copper zone on F.Cu, net VOUT_12V
- added copper zone on F.Cu, net VSS
- added copper zone on F.Cu, net VSYS
