File: power_module_v2alt.kicad_pcb (KiCad board)
At the start: 4 copper layers, 100 x 85 mm, 77 parts, among them J1_BMS1 I2C+ALERT, J1_INPUT1 USB_C_16P, Q1_BMS1 AON7544, Q1_BUCKBOOST1 AON7544, Q2_BMS1 AON7544, Q2_BUCKBOOST1 AON7544, Q3_BUCKBOOST1 AON7544, Q4_BUCKBOOST1 AON7544, SW1_BMS1 Kill Switch, U1_BMS1 BQ7692003PWR, U1_BUCKBOOST1 LM5176PWP, U1_CHARGER1 IP2326, U1_INPUT1 CH224K

Commit message: Fixing remaining disconnects
Parts:
- moved R9_CHARGER1 6.43 mm to (57.9, 6.03), turned to -90 degrees
- moved R10_BMS1 3.60 mm to (83.8, 12.2)
- moved R8_CHARGER1 1.74 mm to (59.4, 5.84)
- moved R7_CHARGER1 1.62 mm to (61.7, 7.62)
- moved R8_BMS1 0.87 mm to (77.5, 51.3)
- moved R3_CHARGER1 0.57 mm to (55.4, 15.4)
Routing:
- net VBUS_RAW: track 43.9 -> 76.1 mm
- net VSET: track 38.8 -> 7.98 mm, vias 0 -> 2
- net VBUS_9V: track 19.8 -> 37.5 mm
- net CHG_EN: track 11.1 -> 2.29 mm
- net LED_K: track 0.00 -> 8.65 mm, vias 0 -> 2
- net REGOUT: track 22.6 -> 30.0 mm
- net GND: track 69.6 -> 75.1 mm, vias 37 -> 40
- net LX_SW: track 3.40 -> 8.73 mm
- net DSG_DRV_GATED: track 14.0 -> 10.7 mm
- net VSS: track 81.1 -> 84.1 mm
- net VSYS: track 23.7 -> 26.6 mm
- net DSG_DRV: track 40.5 -> 39.0 mm
- net CC1: track 18.3 -> 19.6 mm
- net CHG_DRV: track 8.82 -> 7.69 mm
- net BAT+: track 14.1 -> 13.1 mm, vias 9 -> 12
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
Commit message: Oops, forgot to save, apparently
Parts:
- moved R3_BMS1 7.33 mm to (86.9, 53.1)
Routing:
- net VC2: track 16.5 -> 11.6 mm
- net VC3: track 14.0 -> 10.8 mm
Changed lines of the file:
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@@
 	(footprint "Resistor_SMD:R_0603_1608Metric"
 		(layer "F.Cu")
-		(at 79.9763 50.5973 180)
+		(at 86.868 53.086 180)
 		(descr "Resistor SMD 0603 (1608 Metric), square (rectangular) end terminal, IPC-7351 nominal, (Body size source: IPC-SM-782 page 72, https://www.pcb-3d.com/wordpress/wp-content/uploads/ipc-sm-782a_amendment_1_and_2.pdf), generated with kicad-footprint-generator")
 		(tags "resistor")
@@
 	)
 	(segment
-		(start 83.4803 49.8959)
-		(end 81.5027 49.8959)
-		(width 0.2)
-		(layer "F.Cu")
-		(net 5)
-	)
-	(segment
 		(start 86.7705 48.5415)
 		(end 84.8347 48.5415)
@@
 	)
 	(segment
-		(start 81.5027 49.8959)
-		(end 80.8013 50.5973)
-		(width 0.2)
-		(layer "F.Cu")
-		(net 5)
-	)
-	(segment
-		(start 84.8347 48.5415)
-		(end 83.4803 49.8959)
-		(width 0.2)
-		(layer "F.Cu")
-		(net 5)
-	)
-	(segment
 		(start 84.8347 48.5415)
 		(end 84.8347 48.376)
@@
 	)
 	(segment
-		(start 83.155 50.6324)
-		(end 84.775 52.2524)
+		(start 83.2847 49.0493)
+		(end 83.155 49.179)
 		(width 0.2)
 		(layer "F.Cu")
@@
 	(segment
 		(start 83.2847 48.376)
-		(end 81.8176 48.376)
-		(width 0.2)
-		(layer "F.Cu")
-		(net 29)
-	)
-	(segment
-		(start 80.4097 51.3948)
-		(end 82.3926 51.3948)
+		(end 83.2847 49.0493)
 		(width 0.2)
 		(layer "F.Cu")
@@
 	)
 	(segment
-		(start 81.8176 48.376)
-		(end 80.0988 50.0948)
+		(start 83.155 50.6324)
+		(end 84.775 52.2524)
 		(width 0.2)
 		(layer "F.Cu")
@@
 	)
 	(segment
-		(start 80.0988 50.0948)
-		(end 80.0988 51.0839)
+		(start 80.8625 47.275)
+		(end 82.1837 47.275)
 		(width 0.2)
 		(layer "F.Cu")
@@
 	)
 	(segment
-		(start 82.3926 51.3948)
+		(start 83.155 49.179)
 		(end 83.155 50.6324)
 		(width 0.2)
@@
 	)
 	(segment
-		(start 80.0988 51.0839)
-		(end 80.4097 51.3948)
+		(start 82.1837 47.275)
+		(end 83.2847 48.376)
 		(width 0.2)
 		(layer "F.Cu")
